File: runtime.kicad_pcb (KiCad board)
At the start: 2 copper layers, 28.1 x 46 mm, 7 parts, among them U1 AS5600, U2 XIAO-RP2040-DIP

Commit message: fixing ground pour issues
Routing:
- net /GND: track 36.8 -> 0.00 mm, vias 2 -> 0
Changed lines of the file:
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@@
+	)
+	(segment
+		(start 122 95)
+		(end 124.2075 92.7925)
+		(width 0.2)
+		(layer "F.Cu")
+		(net "/GPIO")
+	)
+	(segment
+		(start 122 113)
+		(end 122 95)
+		(width 0.2)
+		(layer "F.Cu")
+		(net "/GPIO")
+	)
+	(segment
+		(start 124.2075 92.7925)
+		(end 124.5875 92.7925)
+		(width 0.2)
+		(layer "F.Cu")
+		(net "/GPIO")
+	)
+	(segment
+		(start 130.629216 127)
+		(end 130.629216 121.629216)
+		(width 0.2)
+		(layer "F.Cu")
+		(net "/GPIO")
+	)
+	(segment
+		(start 130.629216 121.629216)
+		(end 122 113)
+		(width 0.2)
+		(layer "F.Cu")
+		(net "/GPIO")
+	)
+	(segment
+		(start 128.475 105.34)
+		(end 126.0875 102.9525)
+		(width 0.2)
+		(layer "F.Cu")
+		(net "/SDA")
+	)
+	(segment
+		(start 133.16 114)
+		(end 133.525 114.365)
+		(width 0.2)
+		(layer "F.Cu")
+		(net "/SDA")
+	)
+	(segment
+		(start 128.475 114)
+		(end 133.16 114)
+		(width 0.2)
+		(layer "F.Cu")
+		(net "/SDA")
+	)
+	(segment
+		(start 126.0875 102.9525)
+		(end 124.5875 102.9525)
+		(width 0.2)
+		(layer "F.Cu")
+		(net "/SDA")
+	)
+	(segment
+		(start 128.475 114)
+		(end 128.475 105.34)
+		(width 0.2)
+		(layer "F.Cu")
+		(net "/SDA")
 	)
 	(segment
@@
 		(net "/SCL")
 	)
-	(segment
-		(start 128.475 105.34)
-		(end 126.0875 102.9525)
-		(width 0.2)
-		(layer "F.Cu")
-		(net "/SDA")
-	)
-	(segment
-		(start 133.16 114)
-		(end 133.525 114.365)
-		(width 0.2)
-		(layer "F.Cu")
-		(net "/SDA")
-	)
-	(segment
-		(start 128.475 114)
-		(end 133.16 114)
-		(width 0.2)
-		(layer "F.Cu")
-		(net "/SDA")
-	)
-	(segment
-		(start 126.0875 102.9525)
-		(end 124.5875 102.9525)
-		(width 0.2)
-		(layer "F.Cu")
-		(net "/SDA")
-	)
-	(segment
-		(start 128.475 114)
-		(end 128.475 105.34)
-		(width 0.2)
-		(layer "F.Cu")
-		(net "/SDA")
-	)
-	(segment
-		(start 133.870552 116.905)
-		(end 133.525 116.905)
-		(width 0.2)
-		(layer "F.Cu")
-		(net "/GND")
-	)
-	(segment
-		(start 133.525 116.905)
-		(end 133.525 117.525)
-		(width 0.2)
-		(layer "F.Cu")
-		(net "/GND")
-	)
-	(segment
-		(start 137.680552 113.095)
-		(end 133.870552 116.905)
-		(width 0.2)
-		(layer "F.Cu")
-		(net "/GND")
-	)
-	(segment
-		(start 138.475 98.040256)
-		(end 138.475 113.095)
-		(width 0.2)
-		(layer "F.Cu")
-		(net "/GND")
-	)
-	(segment
-		(start 141.182756 95.3325)
-		(end 138.475 98.040256)
-		(width 0.2)
-		(layer "F.Cu")
-		(net "/GND")
-	)
-	(segment
-		(start 134 125.370784)
-		(end 135.629216 127)
-		(width 0.2)
-		(layer "F.Cu")
-		(net "/GND")
-	)
-	(segment
-		(start 138.475 113.095)
-		(end 137.680552 113.095)
-		(width 0.2)
-		(layer "F.Cu")
-		(net "/GND")
-	)
-	(segment
-		(start 141.5875 95.3325)
-		(end 141.182756 95.3325)
-		(width 0.2)
-		(layer "F.Cu")
-		(net "/GND")
-	)
-	(segment
-		(start 134 120)
-		(end 134 125.370784)
-		(width 0.2)
-		(layer "F.Cu")
-		(net "/GND")
-	)
-	(segment
-		(start 133.525 117.525)
-		(end 134 118)
-		(width 0.2)
-		(layer "F.Cu")
-		(net "/GND")
-	)
-	(via
-		(at 134 118)
-		(size 0.6)
-		(drill 0.3)
-		(layers "F.Cu" "B.Cu")
-		(net "/GND")
-	)
-	(via
-		(at 134 120)
-		(size 0.6)
-		(drill 0.3)
-		(layers "F.Cu" "B.Cu")
-		(net "/GND")
-	)
-	(segment
-		(start 134 118)
-		(end 134 120)
-		(width 0.2)
-		(layer "B.Cu")
-		(net "/GND")
-	)
-	(segment
-		(start 122 95)
-		(end 124.2075 92.7925)
-		(width 0.2)
-		(layer "F.Cu")
-		(net "/GPIO")
-	)
-	(segment
-		(start 122 113)
-		(end 122 95)
-		(width 0.2)
-		(layer "F.Cu")
-		(net "/GPIO")
-	)
-	(segment
-		(start 124.2075 92.7925)
-		(end 124.5875 92.7925)
-		(width 0.2)
-		(layer "F.Cu")
-		(net "/GPIO")
-	)
-	(segment
-		(start 130.629216 127)
-		(end 130.629216 121.629216)
-		(width 0.2)
-		(layer "F.Cu")
-		(net "/GPIO")
-	)
-	(segment
-		(start 130.629216 121.629216)
-		(end 122 113)
-		(width 0.2)
-		(layer "F.Cu")
-		(net "/GPIO")
-	)
 	(zone
 		(net "/GND")
@@
 		(hatch edge 0.5)
 		(connect_pads
-			(clearance 0.5)
+			(clearance 0.25)
 		)
 		(min_thickness 0.25)
